Commit message: added camera

File: src/awdbot/awdbot_description/urdf/awdbot.urdf.xacro (robot description, xacro)
@@ -118,4 +118,22 @@
         </visual>
     </link>
+    <link name="camera_link">
+        <xacro:box_inertial name="camera_link" m="${camera_mass}" x="${camera_width}" y="${camera_length}" z="${camera_height}" />
+        <visual>
+            <geometry>
+                <box size="${camera_width} ${camera_length} ${camera_height}"/>
+            </geometry>
+        </visual>
+        <collision>
+            <geometry>
+                <box size="${camera_width} ${camera_length} ${camera_height}" />
+            </geometry>
+        </collision>
+        <inertial>
+            <mass value="0.0"/>
+            <origin xyz="0.0 0.0 0.0" rpy="0.0 0.0 0.0"/>
+            <inertia ixx="0.0" ixy="0.0" ixz="0.0" iyy="0.0" iyz="0.0" izz="0.0"/>
+        </inertial>
+    </link>
     <joint name="wheel_front_right_joint" type="continuous">
         <parent link="base_link" />
@@ -142,4 +160,10 @@
         <axis xyz="0 1 0" />
     </joint>
+    <joint name="camera_joint" type="fixed">
+        <parent link="base_link"/>
+        <child link="camera_link"/>
+        <origin xyz="${chassis_length/2} 0 ${chassis_height/2+camera_height/2}" rpy="0  1.570796327 0"/>
+        <axis xyz="0 0 0"/>
+    </joint>
     <joint name="lidar_joint" type="fixed">
       <parent link="base_link"/>

Commit message: Added opencv package; added light to awdbot

File: src/awdbot/awdbot_description/urdf/awdbot.urdf.xacro (robot description, xacro)
@@ -163,5 +163,5 @@
         <parent link="base_link"/>
         <child link="camera_link"/>
-        <origin xyz="${chassis_length/2} 0 ${chassis_height/2+camera_height/2}" rpy="0  1.570796327 0"/>
+        <origin xyz="${chassis_length/2} 0 ${chassis_height/2+camera_height/2}" rpy="0 1.2 0"/>
         <axis xyz="0 0 0"/>
     </joint>
@@ -172,3 +172,12 @@
       <axis xyz="0 0 1"/>
     </joint>
+    <xacro:include filename="awdbot/light.xacro"/>
+    <xacro:led_strip8_with_lights
+      side="R" parent="base_link"
+      x="${chassis_length/2-0.05}" y="-0.04" z="${chassis_height/2+0.1}" dx="0.01"
+      on_color="1.0 1.0 1.0 1.0" off_color="0.0 0.0 0.0 1.0"
+      light_range="0.5"
+      on0="1" on1="1" on2="1" on3="1" on4="1" on5="1" on6="1" on7="1"
+      light_direction="0 0 0"
+      light_rpy="${-45*3.141/180} 0 ${90*3.141/180}"/>
 </robot>

File: src/awdbot/awdbot_description/urdf/awdbot/awdbot_gazebo.xacro (robot description, xacro)
@@ -163,5 +163,5 @@
         <camera>
             <camera_info_topic>camera/camera_info</camera_info_topic>
-            <horizontal_fov>1.089</horizontal_fov>
+            <horizontal_fov>2.0</horizontal_fov>
             <image>
                 <format>R8G8B8</format>

Commit message: opencv linefollower fertig

File: src/awdbot/awdbot_description/urdf/awdbot.urdf.xacro (robot description, xacro)
@@ -163,5 +163,5 @@
         <parent link="base_link"/>
         <child link="camera_link"/>
-        <origin xyz="${chassis_length/2} 0 ${chassis_height/2+camera_height/2}" rpy="0 1.2 0"/>
+        <origin xyz="${chassis_length/2+0.01} 0 ${chassis_height/2+camera_height/2}" rpy="0 0.8 0"/>
         <axis xyz="0 0 0"/>
     </joint>
